File: design/temp.sch (KiCad schematic (older format))
At the start: 3 parts

Commit message: WIP
Parts:
- C41: symbol C-RESCUE-BLDC_4 -> BLDC_4-rescue:C-RESCUE-BLDC_4
- R1, R2: symbol R-RESCUE-BLDC_4 -> BLDC_4-rescue:R-RESCUE-BLDC_4
Connections:
- wire segments 7 -> 10
Changed lines of the file:
@@
-EESchema Schematic File Version 2
-LIBS:BLDC_4-rescue
-LIBS:power
-LIBS:device
-LIBS:transistors
-LIBS:conn
-LIBS:linear
-LIBS:regul
-LIBS:74xx
-LIBS:cmos4000
-LIBS:adc-dac
-LIBS:memory
-LIBS:xilinx
-LIBS:microcontrollers
-LIBS:dsp
-LIBS:microchip
-LIBS:analog_switches
-LIBS:motorola
-LIBS:texas
-LIBS:intel
-LIBS:audio
-LIBS:interface
-LIBS:digital-audio
-LIBS:philips
-LIBS:display
-LIBS:cypress
-LIBS:siliconi
-LIBS:opto
-LIBS:atmel
-LIBS:contrib
-LIBS:valves
-LIBS:crf_1
+EESchema Schematic File Version 4
 LIBS:BLDC_4-cache
-EELAYER 25 0
+EELAYER 29 0
 EELAYER END
 $Descr A4 11693 8268
 encoding utf-8
-Sheet 3 7
-Title "BLDC Driver 4.11"
-Date "21 aug 2015"
-Rev "4.12"
-Comp "Benjamin Vedder"
+Sheet 3 6
+Title "Low-power BLDC Driver"
+Date "2019-05-11"
+Rev "0.1"
+Comp "Christian Conkle - Benjamin Vedder "
 Comment1 ""
 Comment2 ""
@@
 $EndDescr
 $Comp
-L R-RESCUE-BLDC_4 R1
+L BLDC_4-rescue:R-RESCUE-BLDC_4 R1
 U 1 1 5426DA2F
 P 4400 3400
@@
 $EndComp
 $Comp
-L R-RESCUE-BLDC_4 R2
+L BLDC_4-rescue:R-RESCUE-BLDC_4 R2
 U 1 1 5426DAA6
 P 4400 4100
@@
 $EndComp
 $Comp
-L C-RESCUE-BLDC_4 C41
+L BLDC_4-rescue:C-RESCUE-BLDC_4 C41
 U 1 1 5426DADD
 P 4150 4100
@@
 $EndComp
 $Comp
-L VCC #PWR023
+L power:VCC #PWR023
 U 1 1 5426DB11
 P 4400 3050
@@
 $EndComp
 $Comp
-L GND-RESCUE-BLDC_4 #PWR024
+L BLDC_4-rescue:GND-RESCUE-BLDC_4 #PWR024
 U 1 1 5426DB25
 P 4400 4600
@@
 $EndComp
 Wire Wire Line
-	4400 4350 4400 4600
+	4400 4350 4400 4450
 Wire Wire Line
 	4150 4300 4150 4450
@@
 Connection ~ 4400 4450
 Wire Wire Line
-	4400 3650 4400 3850
+	4400 3650 4400 3750
 Wire Wire Line
-	4150 3750 4550 3750
+	4150 3750 4400 3750
 Wire Wire Line
 	4150 3750 4150 3900
@@
 Text HLabel 4550 3750 2    60   Input ~ 0
 Temp
+Wire Wire Line
+	4400 4450 4400 4600
+Wire Wire Line
+	4400 3750 4400 3850
+Wire Wire Line
+	4400 3750 4550 3750
 $EndSCHEMATC
