File: design/BLDC_4.sch (KiCad schematic (older format))
At the start: 26 parts, among them K1 SERVO, P1 HALL/Encoder, P101 CANBUS, P3 PWR_COMM, P4 IN+, P5 IN-, P6 MOTOR1, P7 MOTOR2, P9 MOTOR3, X1 MINI-USB-SHIELD-32005-201

Commit message: WIP
Parts:
- removed C3: 100n, CRF1:SMD-0603_c, symbol C-RESCUE-BLDC_4
- removed K1: SERVO, CRF1:pinhead-1X03, symbol CONN_3
- removed P1: HALL/Encoder, CRF1:MICRO_JST_6, symbol CONN_6
- removed R5: 2k2, CRF1:SMD-0603_r, symbol R-RESCUE-BLDC_4
- removed R53, R54: SHUNT, CRF1:WSLP2726, symbol SHUNT
- removed R6: 0R, CRF1:SMD-0603_r, symbol R-RESCUE-BLDC_4
- removed X1: MINI-USB-SHIELD-32005-201, CRF1:USB-UX60R-MB-5ST, symbol MINI-USB-SCHIELD-32005-201
- added C14: 2.2u, Capacitor_SMD:C_0805_2012Metric_Pad1.15x1.40mm_HandSolder, symbol BLDC_4-rescue:C-RESCUE-BLDC_4
- added C20, C21: 220u 50V, symbol Device:CP_Small
- added J1: USB_B_Micro, symbol Connector:USB_B_Micro
- added R1: NTC 10k, Resistor_SMD:R_0805_2012Metric_Pad1.15x1.40mm_HandSolder, symbol BLDC_4-rescue:R-RESCUE-BLDC_4
- added R2: 10k, Resistor_SMD:R_0805_2012Metric_Pad1.15x1.40mm_HandSolder, symbol BLDC_4-rescue:R-RESCUE-BLDC_4
- C2: value 100n -> 0.1u 16V; footprint CRF1:SMD-0603_c -> Capacitor_SMD:C_0805_2012Metric_Pad1.15x1.40mm_HandSolder; symbol C-RESCUE-BLDC_4 -> BLDC_4-rescue:C-RESCUE-BLDC_4; digikey# (none) -> 445-6938-1-ND; manf# (none) -> C2012X7R2A104K125AA
- D1, D2, D3: symbol LED-RESCUE-BLDC_4 -> BLDC_4-rescue:LED-RESCUE-BLDC_4
- P101: symbol CONN_4 -> BLDC_4-rescue:CONN_4
- P3: symbol CONN_01X07 -> BLDC_4-rescue:CONN_01X07
- P4, P5, P6, P7, P9: symbol CONN_1 -> BLDC_4-rescue:CONN_1
- R103, R104, R22, R3, R37, R38, R4: footprint CRF1:SMD-0603_r -> Resistor_SMD:R_0805_2012Metric_Pad1.15x1.40mm_HandSolder; symbol R-RESCUE-BLDC_4 -> BLDC_4-rescue:R-RESCUE-BLDC_4
Connections:
- net labels added: GNDPWR
- wire segments 91 -> 87
Other:
- note added: "Voltage supply (0 - 50v)\nNeeds external decoupling\ncaps to avoid high voltage\ntransients produced by the\ninductance of the battery\nwiring while switching the FETs\nAlso critical for EMI/RF compliance"
- note removed: "100R if used as\nservo output"
- note removed: "Connect signal ground and\npower ground in one place only"
- note removed: "Mount 0R if used\nas USB host"
- note removed: "Voltage supply (0 - 60v)\nNeeds external decoupling\ncaps to avoid high voltage\ntransients produced by the\ninductance of the battery\nwiring while switching the FETs\nAlso critical for EMI/RF compliance"
- moved on the sheet: D1, D2, D3, P4, P5, R103, R22, R37, R38

Commit message: WIP
Parts:
- C20, C21: footprint (none) -> Capacitor_THT:CP_Radial_D10.0mm_P5.00mm
- R2: digikey# (none) -> RMCF0805JT10K0CT-ND; digikey-search (none) -> https://www.digikey.com/products/en/resistors/chip-resistor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
- R3: digikey# (none) -> RMCF0805JT39K0CT-ND; digikey-search (none) -> https://www.digikey.com/products/en/resistors/chip-resistor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
Changed lines of the file:
@@
 F 2 "Resistor_SMD:R_0805_2012Metric_Pad1.15x1.40mm_HandSolder" H 2050 2150 60  0001 C CNN
 F 3 "" H 2050 2150 60  0001 C CNN
+F 4 "RMCF0805JT39K0CT-ND" H 0   0   50  0001 C CNN "digikey#"
+F 5 "https://www.digikey.com/products/en/resistors/chip-resistor-surface-mount/52?FV=1c0011%2C1c0002%2C1c00fa%2C1c0003%2C1c0006%2C1c0008%2C400006%2C1f140000%2Cffe00034%2Cmu39kOhms%7C2085%7C0%2Cmu39kOhms%7C2085%7C1&quantity=0&ColumnSort=1000011&page=1&stock=1&pageSize=100" H 0   0   50  0001 C CNN "digikey-search"
 	1    2050 2150
 	0    -1   1    0
@@
 F 2 "Resistor_SMD:R_0805_2012Metric_Pad1.15x1.40mm_HandSolder" V 2880 6800 30  0001 C CNN
 F 3 "" H 2950 6800 30  0000 C CNN
+F 4 "https://www.digikey.com/products/en/resistors/chip-resistor-surface-mount/52?k=&pkeyword=&wrapfilterschooser=1&sv=0&pv16=6&sf=1&FV=1c0011%2C1c0002%2C1c00fa%2C1c0003%2C1c0006%2C1c0008%2C1f140000%2Cffe00034%2Cmu10+kOhms%7C2085&ColumnSort=0&page=1&stock=1&quantity=&pageSize=100" H 0   0   50  0001 C CNN "digikey-search"
+F 5 "RMCF0805JT10K0CT-ND" H 0   0   50  0001 C CNN "digikey#"
 	1    2950 6800
 	0    -1   -1   0
@@
 F 0 "C20" H 8012 1446 50  0000 R CNN
 F 1 "220u 50V" H 8012 1355 50  0000 R CNN
-F 2 "" H 8100 1400 50  0001 C CNN
+F 2 "Capacitor_THT:CP_Radial_D10.0mm_P5.00mm" H 8100 1400 50  0001 C CNN
 F 3 "~" H 8100 1400 50  0001 C CNN
 F 4 "Cbulk" H 0   0   50  0001 C CNN "Identifier"
@@
 F 0 "C21" H 8488 1446 50  0000 L CNN
 F 1 "220u 50V" H 8488 1355 50  0000 L CNN
-F 2 "" H 8400 1400 50  0001 C CNN
+F 2 "Capacitor_THT:CP_Radial_D10.0mm_P5.00mm" H 8400 1400 50  0001 C CNN
 F 3 "~" H 8400 1400 50  0001 C CNN
 F 4 "Cbulk" H 0   0   50  0001 C CNN "Identifier"
