File: design/CAN.sch (KiCad schematic (older format))
At the start: 4 parts, among them U401 SN65HVD232

Commit message: WIP
Parts:
- added NT14: Net-Tie_2, NetTie:NetTie-2_SMD_Pad0.5mm, symbol Device:Net-Tie_2
- C401: footprint CRF1:SMD-0603_c -> Capacitor_SMD:C_0805_2012Metric_Pad1.15x1.40mm_HandSolder; symbol C-RESCUE-BLDC_4 -> BLDC_4-rescue:C-RESCUE-BLDC_4; digikey# (none) -> 445-5157-1-ND; digikey-search (none) -> https://www.digikey.com/products/en/capacitors/ceramic-capa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; manf# (none) -> C1608X5R1C225K080AB
- R401, R402: footprint CRF1:SMD-0603_r -> Resistor_SMD:R_0805_2012Metric_Pad1.15x1.40mm_HandSolder; symbol R-RESCUE-BLDC_4 -> BLDC_4-rescue:R-RESCUE-BLDC_4
- U401: symbol MCP2551-I/SN-RESCUE-BLDC_4 -> BLDC_4-rescue:MCP2551-I_SN-RESCUE-BLDC_4
Connections:
- wire segments 8 -> 13
Other:
- moved on the sheet: C401
Changed lines of the file:
@@
-EESchema Schematic File Version 2
-LIBS:BLDC_4-rescue
-LIBS:power
-LIBS:device
-LIBS:transistors
-LIBS:conn
-LIBS:linear
-LIBS:regul
-LIBS:74xx
-LIBS:cmos4000
-LIBS:adc-dac
-LIBS:memory
-LIBS:xilinx
-LIBS:microcontrollers
-LIBS:dsp
-LIBS:microchip
-LIBS:analog_switches
-LIBS:motorola
-LIBS:texas
-LIBS:intel
-LIBS:audio
-LIBS:interface
-LIBS:digital-audio
-LIBS:philips
-LIBS:display
-LIBS:cypress
-LIBS:siliconi
-LIBS:opto
-LIBS:atmel
-LIBS:contrib
-LIBS:valves
-LIBS:crf_1
+EESchema Schematic File Version 4
 LIBS:BLDC_4-cache
-EELAYER 25 0
+EELAYER 29 0
 EELAYER END
 $Descr A4 11693 8268
 encoding utf-8
-Sheet 4 7
-Title "BLDC Driver 4.11"
-Date "21 aug 2015"
-Rev "4.12"
-Comp "Benjamin Vedder"
+Sheet 2 5
+Title "Low-power BLDC Driver"
+Date "2019-05-11"
+Rev "0.1"
+Comp "Christian Conkle - Benjamin Vedder "
 Comment1 ""
 Comment2 ""
@@
 $EndDescr
 $Comp
-L MCP2551-I/SN-RESCUE-BLDC_4 U401
-U 1 1 53F59F90
-P 5850 4050
-F 0 "U401" H 5600 4350 40  0000 C CNN
-F 1 "SN65HVD232" H 6100 3750 40  0000 C CNN
-F 2 "CRF1:SOIC-8-W" H 5850 4050 35  0001 C CIN
-F 3 "" H 5850 4050 60  0000 C CNN
-	1    5850 4050
-	-1   0    0    -1
-$EndComp
-$Comp
-L GND-RESCUE-BLDC_4 #PWR025
-U 1 1 53F59F97
-P 5850 4450
-F 0 "#PWR025" H 5850 4450 30  0001 C CNN
-F 1 "GND" H 5850 4380 30  0001 C CNN
-F 2 "" H 5850 4450 60  0000 C CNN
-F 3 "" H 5850 4450 60  0000 C CNN
-	1    5850 4450
-	1    0    0    -1
-$EndComp
-$Comp
-L VCC #PWR026
-U 1 1 53F59F9D
-P 5850 3650
-F 0 "#PWR026" H 5850 3750 30  0001 C CNN
-F 1 "VCC" H 5850 3750 30  0000 C CNN
-F 2 "" H 5850 3650 60  0001 C CNN
-F 3 "" H 5850 3650 60  0001 C CNN
-	1    5850 3650
-	1    0    0    -1
-$EndComp
-$Comp
-L C-RESCUE-BLDC_4 C401
+L BLDC_4-rescue:C-RESCUE-BLDC_4 C401
 U 1 1 53F59FA3
-P 6150 3400
-F 0 "C401" H 6150 3500 40  0000 L CNN
-F 1 "2.2u" H 6156 3315 40  0000 L CNN
-F 2 "CRF1:SMD-0603_c" H 6188 3250 30  0001 C CNN
-F 3 "" H 6150 3400 60  0000 C CNN
-	1    6150 3400
-	1    0    0    -1
-$EndComp
-$Comp
-L VCC #PWR027
-U 1 1 53F59FAA
-P 6150 3200
-F 0 "#PWR027" H 6150 3300 30  0001 C CNN
-F 1 "VCC" H 6150 3300 30  0000 C CNN
-F 2 "" H 6150 3200 60  0001 C CNN
-F 3 "" H 6150 3200 60  0001 C CNN
-	1    6150 3200
-	1    0    0    -1
-$EndComp
-$Comp
-L GND-RESCUE-BLDC_4 #PWR028
-U 1 1 53F59FB0
-P 6150 3600
-F 0 "#PWR028" H 6150 3600 30  0001 C CNN
-F 1 "GND" H 6150 3530 30  0001 C CNN
-F 2 "" H 6150 3600 60  0000 C CNN
-F 3 "" H 6150 3600 60  0000 C CNN
-	1    6150 3600
+P 5850 3350
+F 0 "C401" H 5850 3450 40  0000 L CNN
+F 1 "2.2u" H 5856 3265 40  0000 L CNN
+F 2 "Capacitor_SMD:C_0805_2012Metric_Pad1.15x1.40mm_HandSolder" H 5888 3200 30  0001 C CNN
+F 3 "" H 5850 3350 60  0000 C CNN
+F 4 "445-5157-1-ND" H 0   0   50  0001 C CNN "digikey#"
+F 5 "C1608X5R1C225K080AB" H 0   0   50  0001 C CNN "manf#"
+F 6 "https://www.digikey.com/products/en/capacitors/ceramic-capacitors/60?FV=1c0011%2C1c0002%2C1c00fa%2C1c0112%2C1c0003%2C1c0006%2C1c0008%2C380014%2C380016%2C380020%2C380009%2C1f140000%2Cmu2.2%C2%B5F%7C2049%7C0%2Cmu2.2%C2%B5F%7C2049%7C1%2Cffe0003c%2C1437e4&quantity=0&ColumnSort=0&page=1&stock=1&pageSize=100" H 0   0   50  0001 C CNN "digikey-search"
+	1    5850 3350
 	1    0    0    -1
 $EndComp
 $Bitmap
 Pos 8850 4800
-Scale 1,000000
+Scale 1.000000
 Data
 89 50 4E 47 0D 0A 1A 0A 00 00 00 0D 49 48 44 52 00 00 01 8D 00 00 01 8C 08 02 00 00 00 A9 99 69
@@
 0E 79 0A 00 EC 0E 79 0A 00 EC EE D9 FC E8 EC DF DF E2 F1 78 9F 82 01 00 E8 E0 D9 E4 09 6C 06 C8
 3E 46 03 00 20 08 82 61 18 8A E5 1F A2 FF C1 6C 53 00 60 73 A8 4F 01 80 DD FD 0F 13 C8 C1 C2 DB
-BF 08 98 00 00 00 00 49 45 4E 44 AE 42 60 82 00
+BF 08 98 00 00 00 00 49 45 4E 44 AE 42 60 82
 EndData
 $EndBitmap
@@
 CAN_TX
 $Comp
-L R-RESCUE-BLDC_4 R401
+L BLDC_4-rescue:R-RESCUE-BLDC_4 R401
 U 1 1 540030A8
 P 4900 4050
 F 0 "R401" V 4980 4050 40  0000 C CNN
 F 1 "NI" V 4907 4051 40  0000 C CNN
-F 2 "CRF1:SMD-0603_r" V 4830 4050 30  0001 C CNN
+F 2 "Resistor_SMD:R_0805_2012Metric_Pad1.15x1.40mm_HandSolder" V 4830 4050 30  0001 C CNN
 F 3 "" H 4900 4050 30  0000 C CNN
 	1    4900 4050
@@
 CANL
 Wire Wire Line
-	4650 4300 5150 4300
+	4650 4300 4900 4300
 Wire Wire Line
 	5150 4300 5150 4150
@@
 	5150 3950 5150 3800
 Wire Wire Line
-	5150 3800 4650 3800
+	5150 3800 4900 3800
 Connection ~ 4900 3800
 NoConn ~ 6300 4100
 $Comp
-L R-RESCUE-BLDC_4 R402
+L BLDC_4-rescue:R-RESCUE-BLDC_4 R402
 U 1 1 54003136
 P 6400 4600
 F 0 "R402" H 6550 4600 40  0000 C CNN
 F 1 "10k" V 6407 4601 40  0000 C CNN
-F 2 "CRF1:SMD-0603_r" V 6330 4600 30  0001 C CNN
+F 2 "Resistor_SMD:R_0805_2012Metric_Pad1.15x1.40mm_HandSolder" V 6330 4600 30  0001 C CNN
 F 3 "" H 6400 4600 30  0000 C CNN
 	1    6400 4600
@@
 	6400 4250 6300 4250
 $Comp
-L GND-RESCUE-BLDC_4 #PWR029
+L BLDC_4-rescue:GND-RESCUE-BLDC_4 #PWR029
 U 1 1 5400318B
 P 6400 4850
@@
 Text Notes 6450 4750 0    40   ~ 0
 Propagation delay\nresistor
+Wire Wire Line
+	4900 4300 5150 4300
+Wire Wire Line
+	4900 3800 4650 3800
+$Comp
+L power:GND #PWR0135
+U 1 1 5D97DC20
+P 5850 3150
+F 0 "#PWR0135" H 5850 2900 50  0001 C CNN
+F 1 "GND" H 5855 2977 50  0000 C CNN
+F 2 "" H 5850 3150 50  0001 C CNN
+F 3 "" H 5850 3150 50  0001 C CNN
+	1    5850 3150
+	-1   0    0    1
+$EndComp
+$Comp
+L power:VCC #PWR0136
+U 1 1 5D97E1EF
+P 6100 3600
+F 0 "#PWR0136" H 6100 3450 50  0001 C CNN
+F 1 "VCC" V 6117 3728 50  0000 L CNN
+F 2 "" H 6100 3600 50  0001 C CNN
+F 3 "" H 6100 3600 50  0001 C CNN
+	1    6100 3600
+	0    1    1    0
+$EndComp
+$Comp
+L Device:Net-Tie_2 NT14
+U 1 1 5D97E7FA
+P 6000 3600
+F 0 "NT14" H 6000 3781 50  0001 C CNN
+F 1 "Net-Tie_2" H 6000 3690 50  0001 C CNN
+F 2 "NetTie:NetTie-2_SMD_Pad0.5mm" H 6000 3600 50  0001 C CNN
+F 3 "~" H 6000 3600 50  0001 C CNN
+	1    6000 3600
+	1    0    0    -1
+$EndComp
+Wire Wire Line
+	5900 3600 5850 3600
+Wire Wire Line
+	5850 3600 5850 3650
+Wire Wire Line
+	5850 3550 5850 3600
+Connection ~ 5850 3600
+$Comp
+L power:PWR_FLAG #FLG0110
+U 1 1 5D97EC08
+P 5850 3600
+F 0 "#FLG0110" H 5850 3675 50  0001 C CNN
+F 1 "PWR_FLAG" V 5850 3727 50  0001 L CNN
+F 2 "" H 5850 3600 50  0001 C CNN
+F 3 "~" H 5850 3600 50  0001 C CNN
+	1    5850 3600
+	0    -1   -1   0
+$EndComp
+$Comp
+L BLDC_4-rescue:MCP2551-I_SN-RESCUE-BLDC_4 U401
+U 1 1 53F59F90
+P 5850 4050
+F 0 "U401" H 5600 4350 40  0000 C CNN
+F 1 "SN65HVD232" H 6100 3750 40  0000 C CNN
+F 2 "CRF1:SOIC-8-W" H 5850 4050 35  0001 C CIN
+F 3 "" H 5850 4050 60  0000 C CNN
+	1    5850 4050
+	-1   0    0    -1
+$EndComp
+$Comp
+L power:GND #PWR0137
+U 1 1 5D97EE13
+P 5850 4450
+F 0 "#PWR0137" H 5850 4200 50  0001 C CNN
+F 1 "GND" H 5855 4277 50  0000 C CNN
+F 2 "" H 5850 4450 50  0001 C CNN
+F 3 "" H 5850 4450 50  0001 C CNN
+	1    5850 4450
+	1    0    0    -1
+$EndComp
 $EndSCHEMATC

Commit message: WIP
Parts:
- R402: digikey# (none) -> RMCF0805JT10K0CT-ND; digikey-search (none) -> https://www.digikey.com/products/en/resistors/chip-resistor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
- U401: digikey# (none) -> 296-26344-1-ND; manf# (none) -> SN65HVD232DR
Changed lines of the file:
@@
 F 2 "Resistor_SMD:R_0805_2012Metric_Pad1.15x1.40mm_HandSolder" V 6330 4600 30  0001 C CNN
 F 3 "" H 6400 4600 30  0000 C CNN
+F 4 "https://www.digikey.com/products/en/resistors/chip-resistor-surface-mount/52?k=&pkeyword=&wrapfilterschooser=1&sv=0&pv16=6&sf=1&FV=1c0011%2C1c0002%2C1c00fa%2C1c0003%2C1c0006%2C1c0008%2C1f140000%2Cffe00034%2Cmu10+kOhms%7C2085&ColumnSort=0&page=1&stock=1&quantity=&pageSize=100" H 0   0   50  0001 C CNN "digikey-search"
+F 5 "RMCF0805JT10K0CT-ND" H 0   0   50  0001 C CNN "digikey#"
 	1    6400 4600
 	1    0    0    -1
@@
 F 2 "CRF1:SOIC-8-W" H 5850 4050 35  0001 C CIN
 F 3 "" H 5850 4050 60  0000 C CNN
+F 4 "296-26344-1-ND" H 0   0   50  0001 C CNN "digikey#"
+F 5 "SN65HVD232DR" H 0   0   50  0001 C CNN "manf#"
 	1    5850 4050
 	-1   0    0    -1
