File: design/BLDC_4.kicad_pcb (KiCad board)
At the start: 4 copper layers, 38.5 x 65 mm, 127 parts, among them K1 SERVO, P1 HALL/Encoder, P101 CANBUS, P2 SWD, P3 PWR_COMM, P4 IN+, P5 IN-, P6 MOTOR1, P7 MOTOR2, P9 MOTOR3, Q1 IRFS7530, Q2 IRFS7530, Q3 IRFS7530, Q4 IRFS7530, Q5 IRFS7530, Q6 IRFS7530, U1 STM32F40X_LQFP64, U2 TC2117, U3 DRV8302, U401 SN65HVD232, X1 MINI-USB-SHIELD-32005-201, X2 8MHz 10ppm

Commit message: WIP
Parts:
- removed 1PIN (x2): P***, 1pin
- removed 1PIN (x2): P***, Connect:1pin
- removed C18, C20, C23, C24, C26, C52: 2.2u, CRF1:SMD-0603_c
- removed C19: 120p, CRF1:SMD-0603_c
- removed C21: 6.8n, CRF1:SMD-0603_c
- removed C22: 22n, CRF1:SMD-0603_c
- removed C25, C33: 100u, w_smd_cap:c_tant_B
- removed C27, C3: 100n, CRF1:SMD-0603_c
- removed C28, C29, C30: 220n, CRF1:SMD-0603_c
- removed C34, C36: 2.2n, CRF1:SMD-0603_c
- removed C37: 15u,100V, w_smd_cap:c_2220
- removed C39, C40, C43, C44, C49, C8: 10u,50V, CRF1:SMD-1206
- removed C4, C5, C6, C7: 4n7, CRF1:SMD-0603_c
- removed C51: 15u, 100v, w_smd_cap:c_2220
- removed D4: DIODESCH, Diodes_SMD:SMA_Handsoldering
- removed D5: TVS 5V, w_smd_diode:do214ac
- removed G***: oshw_silkscreen-back_3mm, oshw_silkscreen-back_3mm
- removed K1: SERVO, CRF1:pinhead-1X03
- removed L1: 22u, w_smd_inductors:inductor_smd_8x5mm
- removed P1: HALL/Encoder, CRF1:MICRO_JST_6
- removed R11, R12, R13: 2k2, CRF1:SMD-0603_r
- removed R17: 18k, CRF1:SMD-0603_r
- removed R18: 3k3, CRF1:SMD-0603_r
- removed R19: 15k, CRF1:SMD-0603_r
- removed R20, R7, R8: 10k, CRF1:SMD-0603_r
- removed R21: 220k, CRF1:SMD-0603_r
- removed R25: 1M, CRF1:SMD-0603_r
- removed R48, R49, R50, R51: 100R, CRF1:SMD-0603_r
- removed R53, R54: SHUNT, CRF1:WSLP2726
- removed R6: 0R, CRF1:SMD-0603_r
- removed U3: DRV8302, CRF1:TSSOP-56-PP
- removed X1: MINI-USB-SHIELD-32005-201, CRF1:USB-UX60R-MB-5ST
- added NT1: Net-Tie_2, NetTie:NetTie-2_SMD_Pad2.0mm, F.Cu at (246.6, 117.0)
- added NT2: Net-Tie_2, NetTie:NetTie-2_SMD_Pad2.0mm, F.Cu at (246.6, 124.1)
- added NT3: Net-Tie_2, NetTie:NetTie-2_SMD_Pad2.0mm, F.Cu at (246.6, 120.5)
- added NT4: Net-Tie_2, NetTie:NetTie-2_SMD_Pad0.5mm, F.Cu at (244.8, 114.7)
- added NT5: Net-Tie_2, NetTie:NetTie-2_SMD_Pad0.5mm, F.Cu at (237.2, 119.5)
- added NT6: Net-Tie_2, NetTie:NetTie-2_SMD_Pad2.0mm, F.Cu at (195.9, 115.5)
- added NT7: Net-Tie_2, NetTie:NetTie-2_SMD_Pad2.0mm, F.Cu at (203.4, 115.5)
- added NT8: Net-Tie_2, NetTie:NetTie-2_SMD_Pad2.0mm, F.Cu at (195.9, 119.0)
- added NT9: Net-Tie_2, NetTie:NetTie-2_SMD_Pad2.0mm, F.Cu at (195.9, 122.6)
- C1: value 10u,50V -> 1u; footprint CRF1:SMD-1206 -> 0_CWC:C_0805_2012Metric
- C2, C31, D1, D2, D3, P4, P5, Q2, Q4, Q6, R22, R23, R24, R26, R27, R29, R3, R30, R32, R33, R35, R36, R37, R38, R4, R402, R43, R46: moved to F.Cu
- C9: value 10u,50V -> 1u; footprint CRF1:SMD-1206 -> 0_CWC:C_0805_2012Metric; moved to F.Cu
- R10, R9: value 10k -> SHUNT; footprint CRF1:SMD-0603_r -> CRF1:WSLP2726; moved to F.Cu
- R5: value 2k2 -> SHUNT; footprint CRF1:SMD-0603_r -> CRF1:WSLP2726; moved to F.Cu
- U2: value TC2117 -> DRV8323RS; footprint CRF1:SOT-223 -> Package_DFN_QFN:Texas_S-PVQFN-N48_EP5.15x5.15mm_ThermalVias; moved to F.Cu
- moved U2 142.1 mm to (231.0, 118.3), turned to 0 degrees
- moved Q1 140.7 mm to (237.7, 152.4), turned to 90 degrees
- moved C9 132.6 mm to (236.7, 120.4), turned to 270 degrees
- moved Q2 131.6 mm to (234.7, 140.2), turned to 270 degrees
- moved C1 128.6 mm to (225.6, 117.9), turned to 270 degrees
- moved P6 114.0 mm to (171.1, 157.6), turned to 0 degrees
- moved R46 112.1 mm to (201.4, 118.5), turned to 0 degrees
- moved Q6 111.1 mm to (186.2, 141.5), turned to 0 degrees
- moved R43 106.3 mm to (193.9, 128.1), turned to 0 degrees
- moved Q5 102.5 mm to (174.4, 141.5), turned to 0 degrees
- moved R42 101.4 mm to (172.6, 149.5), turned to 0 degrees
- moved P7 100.8 mm to (165.3, 157.6), turned to 0 degrees
- moved R36 96.8 mm to (197.4, 125.6), turned to 0 degrees
- moved R30 94.2 mm to (193.9, 125.6), turned to 0 degrees
- moved Q4 92.7 mm to (186.2, 124.2), turned to 0 degrees
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Connections:
- net /MCU/MISO_ADC_EXT2 renamed /MISO_RX_SCL
- net /MCU/RX_SCL_MOSI renamed /RX_SCL_MOSI
- net /MCU/SCK_ADC_EXT renamed /SCK_ADC_EXT
- net /MCU/TX_SDA_NSS renamed /TX_SDA
- net /MCU/USB_DM renamed /MCU/USB_D-
- net /MCU/USB_DP renamed /MCU/USB_D+
- C1 pad 1: GND -> Net-(C1-Pad1)
- C1 pad 2: V_SUPPLY -> /Mosfet driver/VM_PIN
- C9 pad 1: GND -> Net-(C9-Pad1)
- C9 pad 2: V_SUPPLY -> VCC
- Q2 pad S: /Mosfet driver/H1_LOW -> Net-(Q2-PadS)
- Q4 pad S: GND -> Net-(Q4-PadS)
- Q6 pad S: /Mosfet driver/H3_LOW -> Net-(Q6-PadS)
- R10 pad 1: /Filters/HALL3_IN -> Net-(Q6-PadS)
- R10 pad 2: /Filters/HALL3_OUT -> GNDPWR
- R30 pad 1: /Mosfet driver/H1_LOW -> Net-(Q2-PadS)
- R36 pad 1: /Mosfet driver/H1_LOW -> Net-(Q2-PadS)
- R46 pad 1: /Mosfet driver/H3_LOW -> Net-(Q6-PadS)
- R5 pad 1: /MCU/SERVO -> Net-(Q2-PadS)
- R5 pad 2: Net-(K1-Pad1) -> GNDPWR
- R9 pad 1: /Filters/HALL2_IN -> Net-(Q4-PadS)
- R9 pad 2: /Filters/HALL2_OUT -> GNDPWR
- U1 pad 52: /Filters/HALL3_OUT -> Net-(U1-Pad52)
- U1 pad 57: /MCU/SERVO -> Net-(U1-Pad57)
- U1 pad 58: /Filters/HALL1_OUT -> Net-(U1-Pad58)
- U1 pad 59: /Filters/HALL2_OUT -> Net-(U1-Pad59)
- U1 pad 8: /Filters/TEMP_IN -> /MCU/BR_SO3
- U2 pad 1: GND -> Net-(R6-Pad1)
- U2 pad 2: VCC -> GNDPWR
- U2 pad 3: +5V -> Net-(C4-Pad1)
Routing:
- net GND: track 398.8 -> 0.00 mm, vias 27 -> 1
- net V_SUPPLY: track 290.3 -> 0.00 mm, vias 20 -> 0
- net VCC: track 185.2 -> 2.56 mm, vias 9 -> 0
- net /Mosfet driver/H3_VS: track 166.9 -> 0.00 mm, vias 18 -> 0
- net /Mosfet driver/H1_VS: track 150.6 -> 0.00 mm, vias 17 -> 0
- net /Mosfet driver/H2_VS: track 145.0 -> 0.00 mm, vias 17 -> 0
- net +5V: track 115.3 -> 0.00 mm, vias 4 -> 0
- net /Mosfet driver/H3_LOW: track 53.5 -> 0.00 mm, vias 2 -> 0
- net /Mosfet driver/H1_LOW: track 48.5 -> 0.00 mm, vias 2 -> 0
- net /Mosfet driver/M_H1: track 49.8 -> 1.60 mm, vias 2 -> 0
- net /TX_SDA: track 47.1 -> 0.00 mm, vias 2 -> 0
- net /MCU/ADC_TEMP: track 44.0 -> 0.00 mm
- net /RX_SCL_MOSI: track 41.6 -> 0.00 mm, vias 1 -> 0
- net /Mosfet driver/M_H3: track 40.9 -> 0.00 mm, vias 2 -> 0
- net /MISO_RX_SCL: track 36.0 -> 0.00 mm, vias 1 -> 0
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- removed copper zone on B.Cu, net /Mosfet driver/H1_LOW
- removed copper zone on B.Cu, net /Mosfet driver/H1_VS
- removed copper zone on F.Cu, net /Mosfet driver/H1_VS
- removed copper zone on GND, net /Mosfet driver/H1_VS
- removed copper zone on GND2, net /Mosfet driver/H1_VS
- removed copper zone on B.Cu, net /Mosfet driver/H2_VS
- removed copper zone on F.Cu, net /Mosfet driver/H2_VS
- removed copper zone on GND, net /Mosfet driver/H2_VS
- removed copper zone on GND2, net /Mosfet driver/H2_VS
- removed copper zone on B.Cu, net /Mosfet driver/H3_LOW
- removed copper zone on B.Cu, net /Mosfet driver/H3_VS
- removed copper zone on F.Cu, net /Mosfet driver/H3_VS
- removed copper zone on GND, net /Mosfet driver/H3_VS
- removed copper zone on GND2, net /Mosfet driver/H3_VS
- removed copper zone on B.Cu, net GND
- removed copper zone on F.Cu, net GND
- removed copper zone on GND, net GND
- removed copper zone on GND2, net GND
- removed copper zone on B.Cu, net VCC
- removed copper zone on F.Cu, net V_SUPPLY
Other:
- board outline removed
- board text removed: "Benjamin Vedder"
- board text removed: "H1"
- board text removed: "H2"
- board text removed: "H3"
- board text removed: "MISO"
- board text removed: "MOSI"
- board text removed: "NSS"
- board text removed: "SCK"
- board text removed: "SCL"
- board text removed: "SDA"
- board text removed: "TEMP"
- board text removed: "VESC 4.12"
- board text removed: "vedder.se"

Commit message: WIP
Parts:
- removed C10, C16, C17, C31, C35, C41: 2.2u, CRF1:SMD-0603_c
- removed C15, C38: 15p, CRF1:SMD-0603_c
- removed C32: 100n, CRF1:SMD-0603_c
- removed NT7, NT8, NT9: Net-Tie_2, NetTie:NetTie-2_SMD_Pad2.0mm
- removed R23, R26, R30, R32, R36, R46: 39k, CRF1:SMD-0603_r
- removed R24, R27, R33: 2k2, CRF1:SMD-0603_r
- removed R28, R29, R34, R35, R42, R43: 4R7, CRF1:SMD-0603_r
- removed U1: STM32F40X_LQFP64, CRF1:lqfp64_pad_mod
- removed X2: 8MHz 10ppm, CRF1:Crystal_5x3mm
- added C18: 10u, Capacitor_SMD:C_0805_2012Metric_Pad1.15x1.40mm_HandSolder, F.Cu at (232.2, 70.1)
- added C19: 2.2u 50V, Capacitor_SMD:C_1206_3216Metric_Pad1.42x1.75mm_HandSolder, F.Cu at (262.1, 154.4)
- added C20: 220u 50V, Capacitor_THT:CP_Radial_D10.0mm_P5.00mm, F.Cu at (216.6, 82.7)
- added C21: 220u 50V, Capacitor_THT:CP_Radial_D10.0mm_P5.00mm, F.Cu at (228.4, 82.7)
- added C22: 10u, Capacitor_SMD:C_0805_2012Metric_Pad1.15x1.40mm_HandSolder, F.Cu at (231.5, 67.1)
- added C23: 10u 50V, Capacitor_SMD:C_1206_3216Metric_Pad1.42x1.75mm_HandSolder, F.Cu at (227.4, 60.7)
- added C24: 0.1u 50V, Capacitor_SMD:C_0603_1608Metric_Pad1.05x0.95mm_HandSolder, F.Cu at (262.6, 156.5)
- added C25: 2.2u 50V, Capacitor_SMD:C_1206_3216Metric_Pad1.42x1.75mm_HandSolder, F.Cu at (262.1, 132.1)
- added C26: 0.1u 50V, Capacitor_SMD:C_0603_1608Metric_Pad1.05x0.95mm_HandSolder, F.Cu at (262.6, 130.0)
- added C27: 2.2u 50V, Capacitor_SMD:C_1206_3216Metric_Pad1.42x1.75mm_HandSolder, F.Cu at (262.1, 125.5)
- added C28: 0.1u 50V, Capacitor_SMD:C_0603_1608Metric_Pad1.05x0.95mm_HandSolder, F.Cu at (262.6, 127.5)
- added C3: 0.1u 50V, Capacitor_SMD:C_0603_1608Metric_Pad1.05x0.95mm_HandSolder, F.Cu at (236.7, 72.1)
- added C4: 47n 50V low-ESR, Capacitor_SMD:C_0805_2012Metric_Pad1.15x1.40mm_HandSolder, F.Cu at (232.7, 60.6)
- added C5: 0.1u 16V, Capacitor_SMD:C_0805_2012Metric_Pad1.15x1.40mm_HandSolder, F.Cu at (236.9, 69.4)
- added C6: 1u, Capacitor_SMD:C_0805_2012Metric_Pad1.15x1.40mm_HandSolder, F.Cu at (236.3, 66.5)
- added C7: 2.2u 50V, Capacitor_SMD:C_1206_3216Metric_Pad1.42x1.75mm_HandSolder, F.Cu at (234.7, 137.2)
- added C8: 2.2u 50V, Capacitor_SMD:C_1206_3216Metric_Pad1.42x1.75mm_HandSolder, F.Cu at (232.2, 137.2)
- added D4: D_Schottky_Small_ALT, Diode_SMD:D_PowerDI-123, F.Cu at (216.1, 70.8)
- added L1: 33uH, 100mOhm, Inductor_SMD:L_Bourns-SRU8043, F.Cu at (218.7, 64.0)
- added NT10: Net-Tie_2, NetTie:NetTie-2_SMD_Pad0.5mm, F.Cu at (194.2, 87.1)
- added NT11: Net-Tie_2, NetTie:NetTie-2_SMD_Pad0.5mm, F.Cu at (194.2, 83.0)
- added NT12: Net-Tie_2, NetTie:NetTie-2_SMD_Pad0.5mm, F.Cu at (194.2, 85.0)
- added NT13: Net-Tie_2, NetTie:NetTie-2_SMD_Pad0.5mm, F.Cu at (194.2, 80.9)
- added NT14: Net-Tie_2, NetTie:NetTie-2_SMD_Pad0.5mm, F.Cu at (201.0, 80.9)
- added NT15: Net-Tie_2, NetTie:NetTie-2_SMD_Pad0.5mm, F.Cu at (236.6, 60.1)
- added R11: 2k2, Resistor_SMD:R_0805_2012Metric_Pad1.15x1.40mm_HandSolder, F.Cu at (185.5, 81.4)
- added R12: 39k, Resistor_SMD:R_0805_2012Metric_Pad1.15x1.40mm_HandSolder, F.Cu at (180.8, 84.3)
- added R13: 2k2, Resistor_SMD:R_0805_2012Metric_Pad1.15x1.40mm_HandSolder, F.Cu at (180.8, 81.4)
- added R14: 39k, Resistor_SMD:R_0805_2012Metric_Pad1.15x1.40mm_HandSolder, F.Cu at (180.8, 87.3)
- added R15: 2k2, Resistor_SMD:R_0805_2012Metric_Pad1.15x1.40mm_HandSolder, F.Cu at (185.5, 84.3)
- added R16: 39k, Resistor_SMD:R_0805_2012Metric_Pad1.15x1.40mm_HandSolder, F.Cu at (188.1, 128.0)
- added R6: 8.45k, Resistor_SMD:R_0805_2012Metric_Pad1.15x1.40mm_HandSolder, F.Cu at (226.8, 67.1)
- added R7: 28k, Resistor_SMD:R_0805_2012Metric_Pad1.15x1.40mm_HandSolder, F.Cu at (227.4, 70.1)
- added R8: 100k, Resistor_SMD:R_0805_2012Metric_Pad1.15x1.40mm_HandSolder, F.Cu at (232.7, 63.5)
- C1, C9: footprint 0_CWC:C_0805_2012Metric -> Capacitor_SMD:C_0805_2012Metric_Pad1.15x1.40mm_HandSolder
- C11, C12, C13, C401: footprint CRF1:SMD-0603_c -> Capacitor_SMD:C_0805_2012Metric_Pad1.15x1.40mm_HandSolder
- C14: footprint CRF1:SMD-0603_c -> Capacitor_SMD:C_0805_2012Metric_Pad1.15x1.40mm_HandSolder; moved to F.Cu
- C2: value 100n -> 0.1u 16V; footprint CRF1:SMD-0603_c -> Capacitor_SMD:C_0805_2012Metric_Pad1.15x1.40mm_HandSolder
- NT1, NT2, NT3: footprint NetTie:NetTie-2_SMD_Pad2.0mm -> NetTie:NetTie-2_SMD_Pad0.5mm
- NT6: value Net-Tie_2 -> Net-Tie_8mil; footprint NetTie:NetTie-2_SMD_Pad2.0mm -> CRF1:NetTie-2_SMD_Pad-8mil
- Q1, Q2, Q3, Q4, Q5, Q6: value IRFS7530 -> CSD19531Q5A; footprint CRF1:D2PAK-7-GDS -> Package_TO_SOT_SMD:TDSON-8-1
- R1, R103, R104, R2, R22, R3, R37, R38, R4, R401, R402: footprint CRF1:SMD-0603_r -> Resistor_SMD:R_0805_2012Metric_Pad1.15x1.40mm_HandSolder
- R10, R5, R9: value SHUNT -> R010 1%; footprint CRF1:WSLP2726 -> CRF1:R_2010_Shunt_HandSolder
- moved R5 233.1 mm to (262.1, 149.4), turned to 270 degrees
- moved R9 229.1 mm to (262.1, 137.2), turned to 270 degrees
- moved R10 218.2 mm to (262.1, 120.4), turned to 270 degrees
- moved C14 133.6 mm to (224.9, 89.9), turned to 0 degrees
- moved P9 120.1 mm to (279.4, 149.9), turned to 270 degrees
- moved P7 116.1 mm to (279.4, 135.9), turned to 270 degrees
- moved P6 114.0 mm to (279.4, 121.9), turned to 270 degrees
- moved C13 105.1 mm to (190.3, 87.3), turned to 0 degrees
- moved R2 101.4 mm to (220.2, 89.9), turned to 0 degrees
- moved C12 99.4 mm to (190.3, 84.3), turned to 0 degrees
- moved R1 97.1 mm to (215.4, 89.9)
- moved Q5 95.7 mm to (268.7, 125.5), turned to 180 degrees
- moved Q3 94.7 mm to (268.7, 132.6), turned to 180 degrees
- moved C11 88.8 mm to (185.5, 87.3), turned to 0 degrees
- moved Q6 85.7 mm to (268.7, 118.4)
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Connections:
- net Net-(C1-Pad1) renamed /Mosfet driver/VCP
- C11 pad 2: VCC -> Net-(C11-Pad2)
- C12 pad 2: VCC -> Net-(C12-Pad2)
- C13 pad 2: VCC -> Net-(C13-Pad2)
- C14 pad 1: GND -> /MCU/ADC_TEMP
- C14 pad 2: VCC -> GND
- C401 pad 1: VCC -> GND
- C401 pad 2: GND -> Net-(C401-Pad2)
- NT3 pad 1: Net-(C8-Pad2) -> Net-(C7-Pad1)
- NT3 pad 2: GND -> V_SUPPLY
- P5 pad 1: GND -> GNDPWR
- P6 pad 1: /Mosfet driver/H3_VS -> /MCU/H3_VS
- P7 pad 1: /Mosfet driver/H2_VS -> /MCU/H2_VS
- P9 pad 1: /Mosfet driver/H1_VS -> /MCU/H1_VS
- R10 pad 1: Net-(Q6-PadS) -> Net-(Q6-Pad1)
- R10 pad 2: GNDPWR -> /Mosfet driver/SH3+
- R10 pad 3: /Mosfet driver/SH3+ -> /Mosfet driver/SH3-
- R10 pad 4: /Mosfet driver/SH3- -> GNDPWR
- R5 pad 1: Net-(Q2-PadS) -> Net-(Q2-Pad1)
- R5 pad 2: GNDPWR -> /Mosfet driver/SH1+
- R5 pad 3: /Mosfet driver/SH1+ -> /Mosfet driver/SH1-
- R5 pad 4: /Mosfet driver/SH1- -> GNDPWR
- R9 pad 1: Net-(Q4-PadS) -> GNDPWR
- R9 pad 2: GNDPWR -> /Mosfet driver/SH2-
- R9 pad 4: /Mosfet driver/SH2- -> Net-(Q4-Pad1)
- U2 pad 16: /Mosfet driver/H2_VS -> /MCU/H2_VS
- U2 pad 19: /Mosfet driver/H3_VS -> /MCU/H3_VS
- U2 pad 43: Net-(C8-Pad2) -> GND
- U2 pad 47: V_SUPPLY -> Net-(C7-Pad1)
- U2 pad 9: /Mosfet driver/H1_VS -> /MCU/H1_VS
- U401 pad 3: VCC -> Net-(C401-Pad2)
Routing:
- net /Mosfet driver/M_H1: track 1.60 -> 39.6 mm
- net /MCU/H1_VS: track 0.00 -> 36.2 mm
- net /Mosfet driver/M_H3: track 0.00 -> 32.4 mm
- net /MCU/H3_VS: track 0.00 -> 31.4 mm
- net /Mosfet driver/M_L1: track 0.00 -> 30.2 mm
- net /Mosfet driver/M_H2: track 0.00 -> 28.6 mm
- net /Mosfet driver/M_L3: track 0.00 -> 26.4 mm
- net /MCU/H2_VS: track 0.00 -> 25.5 mm
- net /Mosfet driver/SH3-: track 0.00 -> 24.9 mm, vias 0 -> 2
- net /Mosfet driver/SH1-: track 0.00 -> 24.1 mm, vias 0 -> 2
- net /Mosfet driver/SH1+: track 0.00 -> 23.7 mm, vias 0 -> 2
- net /Mosfet driver/M_L2: track 0.00 -> 23.7 mm
- net /Mosfet driver/SH3+: track 0.00 -> 21.2 mm
- net /Mosfet driver/SH2+: track 0.00 -> 15.9 mm, vias 0 -> 2
- net /Mosfet driver/SH2-: track 0.00 -> 15.7 mm, vias 0 -> 2
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- added copper zone on F.Cu, net Net-(Q4-Pad1)
Other:
- copper layers 4 -> 2
- net class Default: via_dia 0.8 -> 0.6; via_drill 0.5 -> 0.3
- rule via_min_drill: 0.5 -> 0.3
- rule via_min_size: 0.8 -> 0.6

Commit message: WIP
Parts:
- removed NT15, NT4: Net-Tie_2, NetTie:NetTie-2_SMD_Pad0.5mm
- removed R8: 100k, Resistor_SMD:R_0805_2012Metric_Pad1.15x1.40mm_HandSolder
- NT1, NT3: footprint NetTie:NetTie-2_SMD_Pad0.5mm -> NetTie:NetTie-2_SMD_Pad2.0mm
- moved R104 168.8 mm to (201.9, 158.0)
- moved R103 168.8 mm to (204.5, 158.0)
- moved P4 147.1 mm to (249.9, 165.1)
- moved P5 145.5 mm to (238.8, 165.1)
- moved C2 131.2 mm to (205.5, 137.4), turned to 270 degrees
- moved R3 130.1 mm to (203.2, 137.4), turned to 270 degrees
- moved R4 129.0 mm to (207.8, 137.4), turned to 270 degrees
- moved P101 125.5 mm to (189.0, 132.6), turned to 0 degrees
- moved R401 119.6 mm to (189.5, 138.2), turned to 0 degrees
- moved U401 114.1 mm to (189.5, 143.3), turned to 0 degrees
- moved R402 111.7 mm to (184.9, 141.7), turned to 270 degrees
- moved C401 108.2 mm to (189.5, 148.8), turned to 180 degrees
- moved P2 90.2 mm to (206.5, 167.9), turned to 180 degrees
- moved C23 83.9 mm to (242.6, 143.3), turned to 180 degrees
- moved R22 83.1 mm to (195.8, 157.2), turned to 0 degrees
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Connections:
- net Net-(C5-Pad1) renamed /Mosfet driver/SW
- net Net-(Q2-Pad1) renamed /Power MOSFETS/L1_S
- net Net-(Q4-Pad1) renamed /Power MOSFETS/L2_S
- net Net-(Q6-Pad1) renamed /Power MOSFETS/L3_S
- C18 pad 2: Net-(C18-Pad2) -> VCC
- C22 pad 2: Net-(C18-Pad2) -> VCC
- C6 pad 2: Net-(C6-Pad2) -> GND
- C7 pad 1: Net-(C7-Pad1) -> /Mosfet driver/VIN
- C8 pad 1: Net-(C7-Pad1) -> /Mosfet driver/VIN
- L1 pad 2: Net-(C18-Pad2) -> VCC
- NT3 pad 1: Net-(C7-Pad1) -> /Mosfet driver/VIN
- R6 pad 2: GND -> GNDPWR
- U2 pad 35: Net-(C6-Pad2) -> GND
- U2 pad 47: Net-(C7-Pad1) -> /Mosfet driver/VIN
- U2 pad 48: Net-(R8-Pad1) -> /Mosfet driver/VIN
Routing:
- net GNDPWR: track 0.00 -> 65.0 mm, vias 0 -> 61
- net VCC: track 0.00 -> 32.3 mm, vias 0 -> 2
- net /Mosfet driver/VDRAIN: track 0.00 -> 30.9 mm
- net V_SUPPLY: track 0.00 -> 29.6 mm, vias 0 -> 33
- net /Mosfet driver/SW: track 0.00 -> 19.2 mm
- net /Mosfet driver/VIN: track 0.00 -> 14.7 mm
- net /Mosfet driver/VM_PIN: track 0.00 -> 9.34 mm
- net Net-(R6-Pad1): track 0.00 -> 6.06 mm
- net /MCU/ADC_TEMP: track 0.00 -> 5.93 mm
- net Net-(C4-Pad1): track 0.00 -> 4.85 mm
- net GND: track 0.00 -> 4.43 mm
- net Net-(C4-Pad2): track 0.00 -> 4.21 mm
- net /Mosfet driver/VCP: track 0.00 -> 4.00 mm
- net /Mosfet driver/M_H1: track 39.6 -> 35.6 mm
- net Net-(C5-Pad2): track 0.00 -> 3.47 mm
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- added copper zone on F.Cu, net /MCU/H1_VS
- added copper zone on F.Cu, net /MCU/H2_VS
- added copper zone on F.Cu, net /MCU/H3_VS
- added copper zone on F.Cu, net /Mosfet driver/VIN
- added copper zone on F.Cu, net /Mosfet driver/VM_PIN
- added copper zone on F.Cu, net /Power MOSFETS/L1_S
- added copper zone on F.Cu, net /Power MOSFETS/L3_S
- added copper zone on B.Cu, net GNDPWR
- added copper zone on F.Cu, net GNDPWR
- added copper zone on B.Cu, net V_SUPPLY
- added copper zone on F.Cu, net V_SUPPLY
Other:
- board text removed: "CANH"
- board text removed: "CANL"
