File: design/Power.sch (KiCad schematic (older format))
At the start: 48 parts, among them U2 TC2117, U3 DRV8302

Commit message: WIP
Parts:
- removed C1, C39, C40, C43, C44, C49, C8, C9: 10u,50V, CRF1:SMD-1206, symbol C-RESCUE-BLDC_4
- removed C18, C20, C23, C24, C26, C52: 2.2u, CRF1:SMD-0603_c, symbol C-RESCUE-BLDC_4
- removed C19: 120p, CRF1:SMD-0603_c, symbol C-RESCUE-BLDC_4
- removed C21: 6.8n, CRF1:SMD-0603_c, symbol C-RESCUE-BLDC_4
- removed C22: 22n, CRF1:SMD-0603_c, symbol C-RESCUE-BLDC_4
- removed C25, C33: 100u, w_smd_cap:c_tant_B, symbol CP1-RESCUE-BLDC_4
- removed C27: 100n, CRF1:SMD-0603_c, symbol C-RESCUE-BLDC_4
- removed C28, C29, C30: 220n, CRF1:SMD-0603_c, symbol C-RESCUE-BLDC_4
- removed C34, C36: 2.2n, CRF1:SMD-0603_c, symbol C-RESCUE-BLDC_4
- removed C37: 15u,100V, w_smd_cap:c_2220, symbol C-RESCUE-BLDC_4
- removed C51: 15u, 100v, w_smd_cap:c_2220, symbol C-RESCUE-BLDC_4
- removed D4: DIODESCH, Diodes_SMD:SMA_Handsoldering, symbol DIODESCH
- removed D5: TVS 5V, w_smd_diode:do214ac, symbol DIODE
- removed L1: 22u, w_smd_inductors:inductor_smd_8x5mm, symbol INDUCTOR
- removed R17: 18k, CRF1:SMD-0603_r, symbol R-RESCUE-BLDC_4
- removed R18: 3k3, CRF1:SMD-0603_r, symbol R-RESCUE-BLDC_4
- removed R19: 15k, CRF1:SMD-0603_r, symbol R-RESCUE-BLDC_4
- removed R20: 10k, CRF1:SMD-0603_r, symbol R-RESCUE-BLDC_4
- removed R21: 220k, CRF1:SMD-0603_r, symbol R-RESCUE-BLDC_4
- removed R23, R26, R32: 39k, CRF1:SMD-0603_r, symbol R-RESCUE-BLDC_4
- removed R24, R27, R33: 2k2, CRF1:SMD-0603_r, symbol R-RESCUE-BLDC_4
- removed R25: 1M, CRF1:SMD-0603_r, symbol R-RESCUE-BLDC_4
- removed R48, R49, R50, R51: 100R, CRF1:SMD-0603_r, symbol R-RESCUE-BLDC_4
- removed U2: TC2117, CRF1:SOT-223, symbol NCP1117ST33T3G
- removed U3: DRV8302, CRF1:TSSOP-56-PP, symbol DRV8302
- added C1, C6, C9: 1u, Capacitor_SMD:C_0805_2012Metric_Pad1.15x1.40mm_HandSolder, symbol Device:C_Small
- added C18, C22: 10u, Capacitor_SMD:C_0805_2012Metric_Pad1.15x1.40mm_HandSolder, symbol Device:C_Small
- added C23: 10u 50V, symbol Device:CP_Small
- added C3: 0.1u 50V, Capacitor_SMD:C_0603_1608Metric_Pad1.05x0.95mm_HandSolder, symbol Device:C_Small
- added C4: 47n 50V low-ESR, Capacitor_SMD:C_0805_2012Metric_Pad1.15x1.40mm_HandSolder, symbol Device:C_Small
- added C5: 0.1u 16V, Capacitor_SMD:C_0805_2012Metric_Pad1.15x1.40mm_HandSolder, symbol Device:C_Small
- added C7, C8: 2.2u 50V, Capacitor_SMD:C_1206_3216Metric_Pad1.42x1.75mm_HandSolder, symbol Device:C_Small
- added D4: D_Schottky_Small_ALT, Diode_SMD:D_PowerDI-123, symbol Device:D_Schottky_Small_ALT
- added L1: 33uH, 100mOhm, Inductor_SMD:L_Bourns-SRU8043, symbol Device:L
- added NT1, NT15, NT2, NT3, NT4, NT5: Net-Tie_2, NetTie:NetTie-2_SMD_Pad0.5mm, symbol Device:Net-Tie_2
- added R6: 8.45k, Resistor_SMD:R_0805_2012Metric_Pad1.15x1.40mm_HandSolder, symbol Device:R
- added R7: 28k, Resistor_SMD:R_0805_2012Metric_Pad1.15x1.40mm_HandSolder, symbol Device:R
- added R8: 100k, Resistor_SMD:R_0805_2012Metric_Pad1.15x1.40mm_HandSolder, symbol Device:R
- added U2: DRV8323RS, Package_DFN_QFN:Texas_S-PVQFN-N48_EP5.15x5.15mm_ThermalVias, symbol 0_CWC:DRV8323RS
Connections:
- net labels added: BR_SO3, GNDPWR, H1_VS', H2_VS', H3_VS', SCLK, SDI, SDO, SH1+, SH1-, SH2+, SH2-, SH3+, SH3-, VCP, VDRAIN, VM_PIN, nSCS
- net labels removed: +5V, H1_LOW, H2_LOW, H3_LOW, SENS1, SENS2, SENS3, SH1_A, SH1_B, SH2_A, SH2_B
- wire segments 189 -> 65
- no-connect marks 4 -> 1
Other:
- note added: "Power design:\nhttps://webench.ti.com/appinfo/webench/scripts/SDP.cgi?ID=1AADE308087C1594\n\n"
- note removed: "3.3v regulator\nfor the logic"
- note removed: "MCU must sense the\nvoltage at each phase"

Commit message: WIP
Parts:
- C23: footprint (none) -> Capacitor_SMD:C_1206_3216Metric_Pad1.42x1.75mm_HandSolder
- R8: digikey# (none) -> RMCF0805FT100KCT-ND
- U2: digikey# (none) -> 296-47769-1-ND; manf# (none) -> DRV8323RSRGZR
Changed lines of the file:
@@
 F 2 "Resistor_SMD:R_0805_2012Metric_Pad1.15x1.40mm_HandSolder" V 5780 2150 50  0001 C CNN
 F 3 "~" H 5850 2150 50  0001 C CNN
+F 4 "RMCF0805FT100KCT-ND" H 0   0   50  0001 C CNN "digikey#"
 	1    5850 2150
 	-1   0    0    1
@@
 F 2 "Package_DFN_QFN:Texas_S-PVQFN-N48_EP5.15x5.15mm_ThermalVias" H 5250 3500 50  0001 L CNN
 F 3 "" H 5250 3500 50  0001 L CNN
+F 4 "296-47769-1-ND" H 0   0   50  0001 C CNN "digikey#"
+F 5 "DRV8323RSRGZR" H 0   0   50  0001 C CNN "manf#"
 	1    5250 3500
 	1    0    0    -1
@@
 F 0 "C23" H 3513 3046 50  0000 R CNN
 F 1 "10u 50V" H 3513 2955 50  0000 R CNN
-F 2 "" H 3600 3000 50  0001 C CNN
+F 2 "Capacitor_SMD:C_1206_3216Metric_Pad1.42x1.75mm_HandSolder" H 3600 3000 50  0001 C CNN
 F 3 "~" H 3600 3000 50  0001 C CNN
 F 4 "1276-6736-1-ND" H 0   0   50  0001 C CNN "digikey#"

Commit message: WIP
Parts:
- removed NT15, NT4: Net-Tie_2, NetTie:NetTie-2_SMD_Pad0.5mm, symbol Device:Net-Tie_2
- removed R8: 100k, Resistor_SMD:R_0805_2012Metric_Pad1.15x1.40mm_HandSolder, symbol Device:R
- C4: Identifier (none) -> Csw
- NT1, NT3: footprint NetTie:NetTie-2_SMD_Pad0.5mm -> NetTie:NetTie-2_SMD_Pad2.0mm
Connections:
- net GND: now also C6.2, U2.35 (AGND); no longer R6.2
- net GNDPWR: now also R6.2
- net VCC: now also C18.2, C22.2, L1.2
- net VIN: now reaches C7.1, C8.1, NT3.1, U2.47 (VIN)
- net VIN: now also U2.48 (nSHDN)
- net SW: now reaches C5.1, D4.1 (K), L1.1, U2.45 (SW)
Other:
- moved on the sheet: C4
Changed lines of the file:
@@
 	4450 2500 4450 2400
 Wire Wire Line
-	4450 2400 4350 2400
-Wire Wire Line
-	4350 2600 4650 2600
+	4450 2400 4350 2350
+Wire Wire Line
+	4350 2550 4650 2600
 Wire Wire Line
 	3900 2650 4500 2650
@@
 $EndComp
 Wire Wire Line
-	4050 2100 4050 2150
-Wire Wire Line
-	4050 2150 4300 2150
+	4050 2100 4000 2150
+Wire Wire Line
+	4000 2150 4300 2150
 Wire Wire Line
 	4500 2150 4500 2400
-Connection ~ 4050 2150
+Connection ~ 4000 2150
 $Comp
 L power:GND #PWR0109
 U 1 1 5D5FD19B
-P 4050 2350
+P 4000 2350
 AR Path="/504F83BE/5D5FD19B" Ref="#PWR0109"  Part="1"
 AR Path="/5D7BD396/5D5FD19B" Ref="#PWR?"  Part="1"
-F 0 "#PWR0109" H 4050 2100 50  0001 C CNN
-F 1 "GND" V 4055 2222 50  0000 R CNN
-F 2 "" H 4050 2350 50  0001 C CNN
-F 3 "" H 4050 2350 50  0001 C CNN
-	1    4050 2350
+F 0 "#PWR0109" H 4000 2100 50  0001 C CNN
+F 1 "GND" V 4005 2222 50  0000 R CNN
+F 2 "" H 4000 2350 50  0001 C CNN
+F 3 "" H 4000 2350 50  0001 C CNN
+	1    4000 2350
 	0    1    1    0
 $EndComp
@@
 	5850 3600 6300 3600
 Wire Wire Line
-	6300 3600 6300 3500
-Connection ~ 6300 3600
-$Comp
-L power:GND #PWR0110
-U 1 1 5D7B1097
-P 4250 1800
-AR Path="/504F83BE/5D7B1097" Ref="#PWR0110"  Part="1"
-AR Path="/5D7BD396/5D7B1097" Ref="#PWR?"  Part="1"
-F 0 "#PWR0110" H 4250 1550 50  0001 C CNN
-F 1 "GND" V 4255 1672 50  0000 R CNN
-F 2 "" H 4250 1800 50  0001 C CNN
-F 3 "" H 4250 1800 50  0001 C CNN
-	1    4250 1800
-	0    1    1    0
-$EndComp
+	6300 3600 6300 3550
 Wire Wire Line
 	4250 1800 4300 1800
@@
 Wire Wire Line
 	7800 2600 7800 2550
-Connection ~ 7800 2600
-Wire Wire Line
-	7800 2600 7950 2600
 Wire Wire Line
 	7100 2600 7200 2600
@@
 	7350 2600 7350 2750
 Connection ~ 7350 2600
-Wire Wire Line
-	7350 2600 7600 2600
 Wire Wire Line
 	7200 2950 7200 3050
@@
 Text GLabel 5850 1650 0    60   Input ~ 0
 V_SUPPLY
-Wire Wire Line
-	5850 1650 5850 2000
-Wire Wire Line
-	6050 1650 6150 1650
 Wire Wire Line
 	6150 1650 6150 1850
@@
 $EndComp
 $Comp
-L Device:Net-Tie_2 NT15
-U 1 1 5CDBD5E4
-P 7700 2600
-AR Path="/504F83BE/5CDBD5E4" Ref="NT15"  Part="1"
-AR Path="/5D7BD396/5CDBD5E4" Ref="NT?"  Part="1"
-F 0 "NT15" V 7700 2644 50  0001 L CNN
-F 1 "Net-Tie_2" H 7700 2690 50  0001 C CNN
-F 2 "NetTie:NetTie-2_SMD_Pad0.5mm" H 7700 2600 50  0001 C CNN
-F 3 "~" H 7700 2600 50  0001 C CNN
-	1    7700 2600
-	-1   0    0    1
-$EndComp
-$Comp
-L Device:R R8
-U 1 1 5CECF6BF
-P 5850 2150
-AR Path="/504F83BE/5CECF6BF" Ref="R8"  Part="1"
-AR Path="/5D7BD396/5CECF6BF" Ref="R?"  Part="1"
-F 0 "R8" V 5643 2150 50  0000 C CNN
-F 1 "100k" V 5734 2150 50  0000 C CNN
-F 2 "Resistor_SMD:R_0805_2012Metric_Pad1.15x1.40mm_HandSolder" V 5780 2150 50  0001 C CNN
-F 3 "~" H 5850 2150 50  0001 C CNN
-F 4 "RMCF0805FT100KCT-ND" H 0   0   50  0001 C CNN "digikey#"
-	1    5850 2150
-	-1   0    0    1
-$EndComp
-$Comp
 L Device:C_Small C8
 U 1 1 5CF50F0B
@@
 F 0 "NT1" H 3300 2761 50  0001 C CNN
 F 1 "Net-Tie_2" H 3300 2940 50  0001 C CNN
-F 2 "NetTie:NetTie-2_SMD_Pad0.5mm" H 3300 2850 50  0001 C CNN
+F 2 "NetTie:NetTie-2_SMD_Pad2.0mm" H 3300 2850 50  0001 C CNN
 F 3 "~" H 3300 2850 50  0001 C CNN
 	1    3300 2850
-	-1   0    0    1
-$EndComp
-$Comp
-L Device:Net-Tie_2 NT4
-U 1 1 5D756BB9
-P 6400 3600
-AR Path="/504F83BE/5D756BB9" Ref="NT4"  Part="1"
-AR Path="/5D7BD396/5D756BB9" Ref="NT?"  Part="1"
-F 0 "NT4" H 6400 3511 50  0001 C CNN
-F 1 "Net-Tie_2" H 6400 3690 50  0001 C CNN
-F 2 "NetTie:NetTie-2_SMD_Pad0.5mm" H 6400 3600 50  0001 C CNN
-F 3 "~" H 6400 3600 50  0001 C CNN
-	1    6400 3600
 	-1   0    0    1
 $EndComp
@@
 L Device:Net-Tie_2 NT2
 U 1 1 5D5FCD5D
-P 4050 2250
+P 4000 2250
 AR Path="/504F83BE/5D5FCD5D" Ref="NT2"  Part="1"
 AR Path="/5D7BD396/5D5FCD5D" Ref="NT?"  Part="1"
-F 0 "NT2" H 4050 2161 50  0001 C CNN
-F 1 "Net-Tie_2" H 4050 2340 50  0001 C CNN
-F 2 "NetTie:NetTie-2_SMD_Pad0.5mm" H 4050 2250 50  0001 C CNN
-F 3 "~" H 4050 2250 50  0001 C CNN
-	1    4050 2250
+F 0 "NT2" H 4000 2161 50  0001 C CNN
+F 1 "Net-Tie_2" H 4000 2340 50  0001 C CNN
+F 2 "NetTie:NetTie-2_SMD_Pad0.5mm" H 4000 2250 50  0001 C CNN
+F 3 "~" H 4000 2250 50  0001 C CNN
+	1    4000 2250
 	0    -1   -1   0
 $EndComp
@@
 L Device:C_Small C4
 U 1 1 5D22AA19
-P 4350 2500
+P 4350 2450
 AR Path="/504F83BE/5D22AA19" Ref="C4"  Part="1"
 AR Path="/5D7BD396/5D22AA19" Ref="C?"  Part="1"
-F 0 "C4" H 4259 2546 50  0000 R CNN
-F 1 "47n 50V low-ESR" H 4259 2455 50  0000 R CNN
-F 2 "Capacitor_SMD:C_0805_2012Metric_Pad1.15x1.40mm_HandSolder" H 4350 2500 50  0001 C CNN
-F 3 "~" H 4350 2500 50  0001 C CNN
-F 4 "399-8092-1-ND" H 0   0   50  0001 C CNN "digikey#"
-F 5 "https://www.digikey.com/products/en/capacitors/ceramic-capacitors/60?k=&pkeyword=&wrapfilterschooser=1&sv=0&pv16=6&sf=1&FV=1437e4%2C143aba%2C142369%2C1c0011%2C1c0002%2C1c00fa%2C1c0112%2C1c0003%2C1c0006%2C1c0008%2C1f140000%2Cffe0003c%2Cmu0.047%C2%B5F%7C2049&ColumnSort=0&page=1&stock=1&quantity=&pageSize=100" H 0   0   50  0001 C CNN "digikey-search"
-F 6 "C0805C473J3GACTU" H 0   0   50  0001 C CNN "manf#"
-	1    4350 2500
+F 0 "C4" H 4442 2541 50  0000 L CNN
+F 1 "47n 50V low-ESR" H 4442 2450 50  0000 L CNN
+F 2 "Capacitor_SMD:C_0805_2012Metric_Pad1.15x1.40mm_HandSolder" H 4350 2450 50  0001 C CNN
+F 3 "~" H 4350 2450 50  0001 C CNN
+F 4 "399-8092-1-ND" H 0   -50 50  0001 C CNN "digikey#"
+F 5 "https://www.digikey.com/products/en/capacitors/ceramic-capacitors/60?k=&pkeyword=&wrapfilterschooser=1&sv=0&pv16=6&sf=1&FV=1437e4%2C143aba%2C142369%2C1c0011%2C1c0002%2C1c00fa%2C1c0112%2C1c0003%2C1c0006%2C1c0008%2C1f140000%2Cffe0003c%2Cmu0.047%C2%B5F%7C2049&ColumnSort=0&page=1&stock=1&quantity=&pageSize=100" H 0   -50 50  0001 C CNN "digikey-search"
+F 6 "C0805C473J3GACTU" H 0   -50 50  0001 C CNN "manf#"
+F 7 "Csw" H 4442 2359 50  0000 L CNN "Identifier"
+	1    4350 2450
 	1    0    0    -1
 $EndComp
@@
 L Device:Net-Tie_2 NT3
 U 1 1 5CF76FC3
-P 5950 1650
+P 6000 1650
 AR Path="/504F83BE/5CF76FC3" Ref="NT3"  Part="1"
 AR Path="/5D7BD396/5CF76FC3" Ref="NT?"  Part="1"
-F 0 "NT3" V 5950 1694 50  0001 L CNN
-F 1 "Net-Tie_2" H 5950 1740 50  0001 C CNN
-F 2 "NetTie:NetTie-2_SMD_Pad0.5mm" H 5950 1650 50  0001 C CNN
-F 3 "~" H 5950 1650 50  0001 C CNN
-	1    5950 1650
-	-1   0    0    1
+F 0 "NT3" V 6000 1694 50  0001 L CNN
+F 1 "Net-Tie_2" H 6000 1740 50  0001 C CNN
+F 2 "NetTie:NetTie-2_SMD_Pad2.0mm" H 6000 1650 50  0001 C CNN
+F 3 "~" H 6000 1650 50  0001 C CNN
+	1    6000 1650
+	-1   0    0    -1
 $EndComp
 $Comp
@@
 	1    0    0    -1
 $EndComp
+$Comp
+L power:GNDPWR #PWR0110
+U 1 1 5CF0C583
+P 4250 1800
+AR Path="/504F83BE/5CF0C583" Ref="#PWR0110"  Part="1"
+AR Path="/5D7BD396/5CF0C583" Ref="#PWR?"  Part="1"
+F 0 "#PWR0110" H 4250 1600 50  0001 C CNN
+F 1 "GNDPWR" V 4254 1691 50  0000 R CNN
+F 2 "" H 4250 1750 50  0001 C CNN
+F 3 "" H 4250 1750 50  0001 C CNN
+	1    4250 1800
+	0    1    1    0
+$EndComp
+Wire Wire Line
+	5850 2300 5850 2400
+Connection ~ 5850 2400
+Text Label 6150 2300 0    50   ~ 0
+VIN
+Wire Wire Line
+	5900 1650 5850 1650
+Wire Wire Line
+	6100 1650 6150 1650
+Wire Wire Line
+	6100 1650 6100 1850
+Wire Wire Line
+	6100 1850 6150 1850
+Connection ~ 6100 1650
+Wire Wire Line
+	7350 2600 7800 2600
+Connection ~ 7800 2600
+Wire Wire Line
+	7800 2600 7950 2600
+Wire Wire Line
+	6300 3550 6500 3550
+Wire Wire Line
+	6500 3550 6500 3600
+Connection ~ 6300 3550
+Wire Wire Line
+	6300 3550 6300 3500
+Text Label 6400 2600 0    50   ~ 0
+SW
 $EndSCHEMATC
