File: design/STM32F4 64LQFP.sch (KiCad schematic (older format))
At the start: 15 parts, among them P2 SWD, U1 STM32F40X_LQFP64, X2 8MHz 10ppm

Commit message: WIP
Parts:
- removed C11, C12, C13, C14: 2.2u, CRF1:SMD-0603_c, symbol C-RESCUE-BLDC_4
- added C11, C12, C13: 2.2u, Capacitor_SMD:C_0805_2012Metric_Pad1.15x1.40mm_HandSolder, symbol Device:C_Small
- added NT10, NT11, NT12, NT13: Net-Tie_2, NetTie:NetTie-2_SMD_Pad0.5mm, symbol Device:Net-Tie_2
- added R11, R13, R15: 2k2, Resistor_SMD:R_0805_2012Metric_Pad1.15x1.40mm_HandSolder, symbol BLDC_4-rescue:R-RESCUE-BLDC_4
- added R12, R14, R16: 39k, Resistor_SMD:R_0805_2012Metric_Pad1.15x1.40mm_HandSolder, symbol BLDC_4-rescue:R-RESCUE-BLDC_4
- C10: footprint CRF1:SMD-0603_c -> Capacitor_SMD:C_0805_2012Metric_Pad1.15x1.40mm_HandSolder; symbol C-RESCUE-BLDC_4 -> Device:C_Small; digikey# (none) -> 445-5157-1-ND; digikey-search (none) -> https://www.digikey.com/products/en/capacitors/ceramic-capa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; manf# (none) -> C1608X5R1C225K080AB
- C15, C38: footprint CRF1:SMD-0603_c -> Capacitor_SMD:C_0603_1608Metric_Pad1.05x0.95mm_HandSolder; symbol C-RESCUE-BLDC_4 -> BLDC_4-rescue:C-RESCUE-BLDC_4; digikey# (none) -> 399-1051-1-ND; digikey-search (none) -> https://www.digikey.com/products/en/capacitors/ceramic-capa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; manf# (none) -> C0603C150J5GACTU
- C16, C17, C31, C35: footprint CRF1:SMD-0603_c -> Capacitor_SMD:C_0805_2012Metric_Pad1.15x1.40mm_HandSolder; symbol C-RESCUE-BLDC_4 -> BLDC_4-rescue:C-RESCUE-BLDC_4; digikey# (none) -> 445-5157-1-ND; digikey-search (none) -> https://www.digikey.com/products/en/capacitors/ceramic-capa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; manf# (none) -> C1608X5R1C225K080AB
- C32: value 100n -> 0.1u 16V; footprint CRF1:SMD-0603_c -> Capacitor_SMD:C_0805_2012Metric_Pad1.15x1.40mm_HandSolder; symbol C-RESCUE-BLDC_4 -> BLDC_4-rescue:C-RESCUE-BLDC_4; digikey# (none) -> 445-6938-1-ND; manf# (none) -> C2012X7R2A104K125AA
- P2: symbol CONN_6 -> BLDC_4-rescue:CONN_6
- U1: symbol STM32F40X_LQFP64 -> crf_1:STM32F40X_LQFP64
- X2: symbol CRYSTAL_SMD -> BLDC_4-rescue:CRYSTAL_SMD
Connections:
- net labels added: BR_SO3, H1_VS, H2_VS, H3_VS, USB_D+, USB_D-
- net labels removed: HALL_1, HALL_2, HALL_3, SENS1, SENS2, SENS3, SERVO, TEMP_MOTOR, USB_DM, USB_DP
- wire segments 60 -> 87
- no-connect marks 13 -> 17
Other:
- note removed: "Bypass, place next to VDD pins"
- moved on the sheet: C10

Commit message: WIP
Parts:
- R12, R14, R16: digikey# (none) -> RMCF0805JT39K0CT-ND; digikey-search (none) -> https://www.digikey.com/products/en/resistors/chip-resistor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
- U1: digikey# (none) -> 497-17428-ND; digikey-search (none) -> https://www.digikey.com/products/en/integrated-circuits-ics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; manf# (none) -> STM32F401RBT6
- X2: footprint CRF1:Crystal_5x3mm -> Crystal:Crystal_SMD_HC49-SD_HandSoldering; digikey# (none) -> 887-1263-1-ND; digikey-search (none) -> https://www.digikey.com/products/en/crystals-oscillators-re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; manf# (none) -> 9C-8.000MEEJ-T
Changed lines of the file:
@@
 F 0 "X2" H 7750 2140 30  0000 C CNN
 F 1 "8MHz 10ppm" H 7800 1950 30  0000 L CNN
-F 2 "CRF1:Crystal_5x3mm" H 7750 2050 60  0001 C CNN
+F 2 "Crystal:Crystal_SMD_HC49-SD_HandSoldering" H 7750 2050 60  0001 C CNN
 F 3 "" H 7750 2050 60  0000 C CNN
 F 4 "ABM3B-8.0-10-1UT" H 7750 2050 60  0001 C CNN "mfg#"
+F 5 "887-1263-1-ND" H 0   0   50  0001 C CNN "digikey#"
+F 6 "https://www.digikey.com/products/en/crystals-oscillators-resonators/crystals/171?k=&pkeyword=&wrapfilterschooser=1&sv=0&pv7=2&pv1989=0&sf=0&FV=1140003%2C3f40013%2Cmu8MHz%7C2150%2Cffe000ab&ColumnSort=1000011&page=1&stock=1&quantity=1&pageSize=100" H 0   0   50  0001 C CNN "digikey-search"
+F 7 "9C-8.000MEEJ-T" H 0   0   50  0001 C CNN "manf#"
 	1    7750 2050
 	1    0    0    -1
@@
 F 2 "Resistor_SMD:R_0805_2012Metric_Pad1.15x1.40mm_HandSolder" H 2250 2800 60  0001 C CNN
 F 3 "" H 2250 2800 60  0001 C CNN
+F 4 "RMCF0805JT39K0CT-ND" H 0   0   50  0001 C CNN "digikey#"
+F 5 "https://www.digikey.com/products/en/resistors/chip-resistor-surface-mount/52?FV=1c0011%2C1c0002%2C1c00fa%2C1c0003%2C1c0006%2C1c0008%2C400006%2C1f140000%2Cffe00034%2Cmu39kOhms%7C2085%7C0%2Cmu39kOhms%7C2085%7C1&quantity=0&ColumnSort=1000011&page=1&stock=1&pageSize=100" H 0   0   50  0001 C CNN "digikey-search"
 	1    2250 2800
 	0    -1   -1   0
@@
 F 2 "Resistor_SMD:R_0805_2012Metric_Pad1.15x1.40mm_HandSolder" H 2250 2300 60  0001 C CNN
 F 3 "" H 2250 2300 60  0001 C CNN
+F 4 "RMCF0805JT39K0CT-ND" H 0   0   50  0001 C CNN "digikey#"
+F 5 "https://www.digikey.com/products/en/resistors/chip-resistor-surface-mount/52?FV=1c0011%2C1c0002%2C1c00fa%2C1c0003%2C1c0006%2C1c0008%2C400006%2C1f140000%2Cffe00034%2Cmu39kOhms%7C2085%7C0%2Cmu39kOhms%7C2085%7C1&quantity=0&ColumnSort=1000011&page=1&stock=1&pageSize=100" H 0   0   50  0001 C CNN "digikey-search"
 	1    2250 2300
 	0    -1   -1   0
@@
 F 2 "Resistor_SMD:R_0805_2012Metric_Pad1.15x1.40mm_HandSolder" H 2250 1850 60  0001 C CNN
 F 3 "" H 2250 1850 60  0001 C CNN
+F 4 "RMCF0805JT39K0CT-ND" H 0   0   50  0001 C CNN "digikey#"
+F 5 "https://www.digikey.com/products/en/resistors/chip-resistor-surface-mount/52?FV=1c0011%2C1c0002%2C1c00fa%2C1c0003%2C1c0006%2C1c0008%2C400006%2C1f140000%2Cffe00034%2Cmu39kOhms%7C2085%7C0%2Cmu39kOhms%7C2085%7C1&quantity=0&ColumnSort=1000011&page=1&stock=1&pageSize=100" H 0   0   50  0001 C CNN "digikey-search"
 	1    2250 1850
 	0    -1   -1   0
@@
 F 2 "CRF1:lqfp64_pad_mod" H 5750 3900 60  0001 C CNN
 F 3 "" H 5750 3900 60  0001 C CNN
+F 4 "497-17428-ND" H 0   0   50  0001 C CNN "digikey#"
+F 5 "https://www.digikey.com/products/en/integrated-circuits-ics/embedded-microcontrollers/685?k=STM32F40&k=&pkeyword=STM32F40&wrapfilterschooser=0&sv=0&pv16=1120&sf=1&FV=ffe002ad%2C1c0011%2C1c0002&ColumnSort=1000011&page=1&stock=1&quantity=1&pageSize=100" H 0   0   50  0001 C CNN "digikey-search"
+F 6 "STM32F401RBT6" H 0   0   50  0001 C CNN "manf#"
 	1    5750 3900
 	1    0    0    -1
