File: design/mosfets.sch (KiCad schematic (older format))
At the start: 15 parts, among them Q1 IRFS7530, Q2 IRFS7530, Q3 IRFS7530, Q4 IRFS7530, Q5 IRFS7530, Q6 IRFS7530

Commit message: WIP
Parts:
- added C19, C25, C27: 2.2u 50V, Capacitor_SMD:C_1206_3216Metric_Pad1.42x1.75mm_HandSolder, symbol Device:C_Small
- added C24, C26, C28: 0.1u 50V, Capacitor_SMD:C_0603_1608Metric_Pad1.05x0.95mm_HandSolder, symbol Device:C_Small
- added NT6, NT7, NT8, NT9: Net-Tie_2, NetTie:NetTie-2_SMD_Pad0.5mm, symbol Device:Net-Tie_2
- added R10, R5, R9: SHUNT, CRF1:WSLP2726, symbol crf_1:SHUNT
- Q1, Q2, Q3, Q4, Q5, Q6: symbol MOSFET_N -> BLDC_4-rescue:MOSFET_N
- R28, R29, R30, R34, R35, R36, R42, R43, R46: footprint CRF1:SMD-0603_r -> Resistor_SMD:R_0805_2012Metric_Pad1.15x1.40mm_HandSolder; symbol R-RESCUE-BLDC_4 -> BLDC_4-rescue:R-RESCUE-BLDC_4
Connections:
- net V_SUPPLY: now also NT7.1, NT8.1, NT9.1; no longer Q1.D, Q3.D, Q5.D
- net H1_LOW: no longer names the net of Q2.S, R30.1, R36.1
- net H1_LOW: now also R5.1
- net H2_LOW: no longer names the net of Q4.S
- net H2_LOW: now also R9.1
- net H3_LOW: no longer names the net of Q6.S, R46.1
- net H3_LOW: now also R10.1
- new net: C19.2, C24.2, NT6.2, NT7.2, Q1.D
- new net: C25.2, C26.2, NT8.2, Q3.D
- new net: C27.2, C28.2, NT9.2, Q5.D
- new net GNDPWR: C19.1, C24.1, C25.1, C26.1, C27.1, C28.1, R10.2, R5.2, R9.2
- new net SH1+: R5.3
- new net SH1-: R5.4
- new net SH2+: R9.3
- new net SH2-: R9.4
- new net SH3+: R10.3
- new net SH3-: R10.4
- new net VDRAIN: NT6.1
Other:
- moved on the sheet: R34, R42

Commit message: WIP
Parts:
- removed NT7, NT8, NT9: Net-Tie_2, NetTie:NetTie-2_SMD_Pad0.5mm, symbol Device:Net-Tie_2
- removed Q1, Q2, Q3, Q4, Q5, Q6: IRFS7530, CRF1:D2PAK-7-GDS, symbol BLDC_4-rescue:MOSFET_N
- removed R28, R29, R34, R35, R42, R43: 4R7, Resistor_SMD:R_0805_2012Metric_Pad1.15x1.40mm_HandSolder, symbol BLDC_4-rescue:R-RESCUE-BLDC_4
- removed R30, R36, R46: 39k, Resistor_SMD:R_0805_2012Metric_Pad1.15x1.40mm_HandSolder, symbol BLDC_4-rescue:R-RESCUE-BLDC_4
- removed R5, R9: SHUNT, CRF1:WSLP2726, symbol crf_1:SHUNT
- added Q1, Q2, Q3, Q4, Q5, Q6: CSD19531Q5A, Package_TO_SOT_SMD:TDSON-8-1, symbol Transistor_FET:CSD19531Q5A
- added R5, R9: R010 1%, CRF1:R_2010_Shunt_HandSolder, symbol Device:R_Shunt
- NT6: value Net-Tie_2 -> Net-Tie_8mil; footprint NetTie:NetTie-2_SMD_Pad0.5mm -> CRF1:NetTie-2_SMD_Pad-8mil
- R10: value SHUNT -> R010 1%; footprint CRF1:WSLP2726 -> CRF1:R_2010_Shunt_HandSolder; symbol crf_1:SHUNT -> Device:R_Shunt; digikey-search (none) -> https://www.digikey.com/products/en/resistors/chip-resistor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
Connections:
- wire segments 74 -> 54

Commit message: WIP
Connections:
- net labels added: L1_S, L2_S, L3_S
Changed lines of the file:
@@
 Wire Wire Line
 	4900 4850 4750 4850
+Text Label 5050 4250 0    50   ~ 0
+L1_S
+Text Label 6600 4250 0    50   ~ 0
+L2_S
+Text Label 8200 4250 0    50   ~ 0
+L3_S
 $EndSCHEMATC
